Commit message: edit readme and get started on robot urdf

File: urdf/robot.urdf.xacro (robot description, xacro)
@@ -13,4 +13,22 @@
     </inertial>
   </xacro:macro>
+  <xacro:property name="robot_width" value = "${0.75}"/>
+  <xacro:property name="robot_length" value = "${0.75}"/>
+<link name="base_link">
+    <visual>
+      <geometry>
+        <box size = "${robot_width} ${robot_length} 0.2"/>
+      </geometry>
+      <material name = "white"/>
+      <origin xyz = "0 0 0" rpy = "0 0 0"/>
+    </visual>
+    <collision>
+      <geometry>
+        <box size = "${robot_width} ${robot_length} 0.2"/>
+      </geometry>
+      <origin xyz = "0 0 0" rpy = "0 0 0"/>
+    </collision>
+    <xacro:default_inertial mass="8"/>
+  </link>
   <gazebo>
     <plugin name="gazebo_ros_control" filename="libgazebo_ros_control.so">

Commit message: add ros2d2 urdf and wpilib diffdrive example

File: urdf/robot.urdf.xacro (robot description, xacro)
@@ -31,4 +31,28 @@
     <xacro:default_inertial mass="8"/>
   </link>
+  <link name="right_front_wheel">
+    <visual>
+      <geometry>
+        <cylinder radius = "0.075" length = "0.05"/>
+      </geometry>
+      <material name = "white"/>
+      <origin rpy="${pi/2} 0 0"/>
+    </visual>
+    <collision>
+     <geometry>
+        <cylinder radius = "0.075" length = "0.05"/>
+      </geometry>
+      <origin rpy="${pi/2} ${pi/2} 0"/>
+    </collision>
+    <xacro:default_inertial mass="1"/>
+  </link>
+  <joint name="right_front_wheel_joint" type="continuous">
+    <parent link="base_link"/>
+    <child link="right_front_wheel"/>
+    <origin xyz = "1 1 0"/>
+    <axis xyz ="0 0 0"/>
+    <limit effort="30" velocity="100"/>
+    <dynamics damping="0.0" friction="0.0"/>
+  </joint>
   <gazebo>
     <plugin name="gazebo_ros_control" filename="libgazebo_ros_control.so">
