Commit message: got body to load in gazebo

File: my_robot/robot.urdf (robot description, URDF)
Before this commit: robot onshape, 5 links, 4 joints
Links:
- link robot_body: geometry collision mesh filename=package://frc_ros_sim/my_robot/robot_body.stl; visual mesh filename=package://frc_ros_sim/my_robot/robot_body.stl
- link wheel: geometry collision mesh filename=package://frc_ros_sim/my_robot/wheel.stl; visual mesh filename=package://frc_ros_sim/my_robot/wheel.stl
- link wheel_2: geometry collision mesh filename=package://frc_ros_sim/my_robot/wheel.stl; visual mesh filename=package://frc_ros_sim/my_robot/wheel.stl
- link wheel_3: geometry collision mesh filename=package://frc_ros_sim/my_robot/wheel.stl; visual mesh filename=package://frc_ros_sim/my_robot/wheel.stl
- link wheel_4: geometry collision mesh filename=package://frc_ros_sim/my_robot/wheel.stl; visual mesh filename=package://frc_ros_sim/my_robot/wheel.stl
Joints:
- joint wheelLeftBack_speed: type revolute -> continuous
- joint wheelLeftFront_speed: type revolute -> continuous
- joint wheelRightBack_speed: type revolute -> continuous
- joint wheelRightFront_speed: type revolute -> continuous
