Commit message: whole robot loads in rviz

File: my_robot/robot.urdf.xacro (robot description, xacro)
@@ -1,4 +1,5 @@
-<robot name="onshape">
-<link name="robot_body">
+<?xml version="1.0"?>
+<robot name="onshape" xmlns:xacro="http://ros.org/wiki/xacro">
+<link name="base_link">
 <visual>
 <origin xyz="0.0185107 -0.0366209 -0.0384443" rpy="0 -0 0" />
@@ -52,5 +53,5 @@
 <joint name="wheelRightBack_speed" type="continuous">
 <origin xyz="0.346811 -0.32092 -0.0130443" rpy="-1.5708 -0 -1.5708" />
-<parent link="robot_body" />
+<parent link="base_link" />
 <child link="wheel" />
 <axis xyz="0 0 1"/>
@@ -85,5 +86,5 @@
 <joint name="wheelRightFront_speed" type="continuous">
 <origin xyz="0.346811 0.0750801 -0.0130443" rpy="-1.5708 -0 -1.5708" />
-<parent link="robot_body" />
+<parent link="base_link" />
 <child link="wheel_2" />
 <axis xyz="0 0 1"/>
@@ -118,5 +119,5 @@
 <joint name="wheelLeftFront_speed" type="continuous">
 <origin xyz="-0.368589 0.0750801 -0.0130443" rpy="-3.14159 -1.5708 0" />
-<parent link="robot_body" />
+<parent link="base_link" />
 <child link="wheel_3" />
 <axis xyz="0 0 1"/>
@@ -151,5 +152,5 @@
 <joint name="wheelLeftBack_speed" type="continuous">
 <origin xyz="-0.368589 -0.32092 -0.0130443" rpy="-1.5708 -0 -1.5708" />
-<parent link="robot_body" />
+<parent link="base_link" />
 <child link="wheel_4" />
 <axis xyz="0 0 1"/>

Commit message: robot loads into gazebo with controllers

File: my_robot/robot.urdf.xacro (robot description, xacro)
@@ -59,4 +59,13 @@
 <joint_properties friction="0.0"/>
 </joint>
+<transmission name="wheelRightBack_speed_trans">
+      <type>transmission_interface/SimpleTransmission</type>
+      <actuator name="wheelRightBack_speed_motor">
+        <mechanicalReduction>1</mechanicalReduction>
+      </actuator>
+      <joint name="wheelRightBack_speed">
+        <hardwareInterface>VelocityJointInterface</hardwareInterface>
+      </joint>
+</transmission>
 <link name="wheel_2">
 <visual>
@@ -92,4 +101,13 @@
 <joint_properties friction="0.0"/>
 </joint>
+<transmission name="wheelRightFront_speed_trans">
+      <type>transmission_interface/SimpleTransmission</type>
+      <actuator name="wheelRightFront_speed_motor">
+        <mechanicalReduction>1</mechanicalReduction>
+      </actuator>
+      <joint name="wheelRightFront_speed">
+        <hardwareInterface>VelocityJointInterface</hardwareInterface>
+      </joint>
+</transmission>
 <link name="wheel_3">
 <visual>
@@ -125,4 +143,13 @@
 <joint_properties friction="0.0"/>
 </joint>
+<transmission name="wheelLeftFront_speed_trans">
+      <type>transmission_interface/SimpleTransmission</type>
+      <actuator name="wheelLeftFront_speed_motor">
+        <mechanicalReduction>1</mechanicalReduction>
+      </actuator>
+      <joint name="wheelLeftFront_speed">
+        <hardwareInterface>VelocityJointInterface</hardwareInterface>
+      </joint>
+</transmission>
 <link name="wheel_4">
 <visual>
@@ -158,4 +185,13 @@
 <joint_properties friction="0.0"/>
 </joint>
+<transmission name="wheelLeftBack_speed_trans">
+      <type>transmission_interface/SimpleTransmission</type>
+      <actuator name="wheelLeftBack_speed_motor">
+        <mechanicalReduction>1</mechanicalReduction>
+      </actuator>
+      <joint name="wheelLeftBack_speed">
+        <hardwareInterface>VelocityJointInterface</hardwareInterface>
+      </joint>
+</transmission>
 <gazebo>
     <plugin name="gazebo_ros_control" filename="libgazebo_ros_control.so">

Commit message: robot drives!

File: my_robot/robot.urdf.xacro (robot description, xacro)
@@ -56,5 +56,5 @@
 <child link="wheel" />
 <axis xyz="0 0 1"/>
-<limit effort="1" velocity="20" />
+<limit effort="30" velocity="20" />
 <joint_properties friction="0.0"/>
 </joint>
@@ -98,5 +98,5 @@
 <child link="wheel_2" />
 <axis xyz="0 0 1"/>
-<limit effort="1" velocity="20" />
+<limit effort="30" velocity="20" />
 <joint_properties friction="0.0"/>
 </joint>
@@ -140,5 +140,5 @@
 <child link="wheel_3" />
 <axis xyz="0 0 1"/>
-<limit effort="1" velocity="20" />
+<limit effort="30" velocity="20" />
 <joint_properties friction="0.0"/>
 </joint>
@@ -182,5 +182,5 @@
 <child link="wheel_4" />
 <axis xyz="0 0 1"/>
-<limit effort="1" velocity="20" />
+<limit effort="30" velocity="20" />
 <joint_properties friction="0.0"/>
 </joint>

Commit message: setup websocket sim launch file

File: my_robot/robot.urdf.xacro (robot description, xacro)
@@ -56,5 +56,5 @@
 <child link="wheel" />
 <axis xyz="0 0 1"/>
-<limit effort="30" velocity="20" />
+<limit effort="30" velocity="70" />
 <joint_properties friction="0.0"/>
 </joint>
@@ -98,5 +98,5 @@
 <child link="wheel_2" />
 <axis xyz="0 0 1"/>
-<limit effort="30" velocity="20" />
+<limit effort="30" velocity="70" />
 <joint_properties friction="0.0"/>
 </joint>
@@ -140,5 +140,5 @@
 <child link="wheel_3" />
 <axis xyz="0 0 1"/>
-<limit effort="30" velocity="20" />
+<limit effort="30" velocity="70" />
 <joint_properties friction="0.0"/>
 </joint>
@@ -182,5 +182,5 @@
 <child link="wheel_4" />
 <axis xyz="0 0 1"/>
-<limit effort="30" velocity="20" />
+<limit effort="30" velocity="70" />
 <joint_properties friction="0.0"/>
 </joint>

Commit message: robot go vroom (incorrectly)

File: my_robot/robot.urdf.xacro (robot description, xacro)
@@ -56,5 +56,5 @@
 <child link="wheel" />
 <axis xyz="0 0 1"/>
-<limit effort="30" velocity="70" />
+<limit effort="200" velocity="200" />
 <joint_properties friction="0.0"/>
 </joint>
@@ -98,5 +98,5 @@
 <child link="wheel_2" />
 <axis xyz="0 0 1"/>
-<limit effort="30" velocity="70" />
+<limit effort="200" velocity="200" />
 <joint_properties friction="0.0"/>
 </joint>
@@ -140,5 +140,5 @@
 <child link="wheel_3" />
 <axis xyz="0 0 1"/>
-<limit effort="30" velocity="70" />
+<limit effort="200" velocity="200" />
 <joint_properties friction="0.0"/>
 </joint>
@@ -182,5 +182,5 @@
 <child link="wheel_4" />
 <axis xyz="0 0 1"/>
-<limit effort="30" velocity="70" />
+<limit effort="200" velocity="200" />
 <joint_properties friction="0.0"/>
 </joint>

Commit message: mass tweaks

File: my_robot/robot.urdf.xacro (robot description, xacro)
@@ -22,5 +22,6 @@
 <inertial>
 <origin xyz="-0.0108892 -0.120946 0.0878113" rpy="0 0 0"/>
-<mass value="285.257" />
+<mass value="85.3592" />
+<!-- <mass value="285.257" /> -->
 <inertia ixx="11.6146" ixy="6.06475e-16"  ixz="3.1135e-16" iyy="11.1779" iyz="-0.0839813" izz="19.7311" />
 </inertial>
